File: ADC/ADC.kicad_pcb (KiCad board)
At the start: 2 copper layers, 38.1 x 63.5 mm, 98 parts, among them P1 CONN_02X05, P2 CONN_02X08, U1 MICA, U2 MICB, U3 TL074, U4 MICC, U5 MICD, U6 AK5703

Commit message: Expanded board, all files
Parts:
- moved C30 35.7 mm to (94.0, 121.9)
- moved R32 35.7 mm to (91.4, 121.9)
- moved R37 33.3 mm to (66.0, 123.2)
- moved R34 26.9 mm to (88.9, 121.9), turned to 90 degrees
- moved C39 26.4 mm to (66.0, 133.3), turned to 90 degrees
- moved R24 24.2 mm to (111.8, 118.1), turned to 270 degrees
- moved C14 24.0 mm to (87.6, 104.1)
- moved R16 24.0 mm to (87.6, 106.7)
- moved R39 22.7 mm to (66.0, 128.3), turned to 270 degrees
- moved R4 21.9 mm to (71.1, 113.0), turned to 90 degrees
- moved C10 21.6 mm to (87.6, 101.6), turned to 180 degrees
- moved D5 21.3 mm to (96.5, 161.3)
- moved C5 20.1 mm to (73.7, 113.0), turned to 90 degrees
- moved C34 19.1 mm to (104.1, 137.2), turned to 90 degrees
- moved C35 18.8 mm to (81.3, 138.4)
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Other:
- board size 38.1 x 63.5 mm -> 48.3 x 63.5 mm
- net class Default: clearance 0.2 -> 0.1524; trace_width 0.25 -> 0.1524; via_dia 0.6 -> 0.3556; via_drill 0.4 -> 0.3302
- rule trace_clearance: 0.2 -> 0.1524
- rule trace_min: 0.2 -> 0.1524
- rule via_min_drill: 0.3 -> 0.3302
- rule via_min_size: 0.4 -> 0.3556

Commit message: Added plot files
Parts:
- added REF**: MountingHole_3mm, Mounting_Holes:MountingHole_3mm, F.Cu at (110.5, 161.3)
- added REF**: MountingHole_3mm, Mounting_Holes:MountingHole_3mm, F.Cu at (77.5, 161.3)
- added REF**: , Mounting_Holes:MountingHole_3mm, F.Cu at (77.5, 102.9)
- added REF**: MountingHole_2-5mm, Mounting_Holes:MountingHole_2-5mm, F.Cu at (123.2, 97.8)
- added REF**: MountingHole_3mm, Mounting_Holes:MountingHole_3mm, F.Cu at (110.5, 102.9)
- moved C30 35.7 mm to (96.5, 157.5)
- moved R32 35.7 mm to (94.0, 157.5)
- moved R37 33.3 mm to (76.2, 154.9)
- moved R34 26.9 mm to (92.7, 148.6), turned to 0 degrees
- moved C39 26.4 mm to (87.6, 148.6), turned to 0 degrees
- moved R24 24.2 mm to (87.6, 116.8), turned to 0 degrees
- moved C14 24.0 mm to (108.0, 116.8)
- moved R16 24.0 mm to (108.0, 119.4)
- moved R39 22.7 mm to (76.2, 108.0), turned to 90 degrees
- moved R4 21.9 mm to (92.7, 109.2), turned to 0 degrees
- moved C10 21.6 mm to (102.9, 116.8), turned to 0 degrees
- moved D5 21.3 mm to (90.2, 141.0)
- moved C5 20.1 mm to (92.7, 106.7), turned to 0 degrees
- moved C34 19.1 mm to (85.1, 135.9), turned to 180 degrees
- moved C35 18.8 mm to (97.8, 147.3)
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Routing:
- net GNDA: track 0.00 -> 296.8 mm, vias 0 -> 2
- net VAA: track 0.00 -> 176.6 mm, vias 0 -> 4
- net +3V3: track 0.00 -> 129.9 mm, vias 0 -> 1
- net VCC: track 0.00 -> 84.0 mm, vias 0 -> 1
- net Net-(C22-Pad1): track 0.00 -> 81.5 mm
- net Net-(C20-Pad1): track 0.00 -> 73.3 mm, vias 0 -> 3
- net Net-(C24-Pad2): track 0.00 -> 63.0 mm, vias 0 -> 2
- net PDN: track 0.00 -> 48.3 mm, vias 0 -> 2
- net Net-(C23-Pad1): track 0.00 -> 48.2 mm
- net L2ch: track 0.00 -> 45.5 mm, vias 0 -> 1
- net CAD0: track 0.00 -> 45.3 mm, vias 0 -> 1
- net SDA: track 0.00 -> 45.1 mm
- net R1ch: track 0.00 -> 44.8 mm
- net Net-(C21-Pad1): track 0.00 -> 44.6 mm
- net Net-(C31-Pad1): track 0.00 -> 42.9 mm
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Other:
- board size 48.3 x 63.5 mm -> 38.1 x 63.5 mm
- net class Default: via_dia 0.3556 -> 0.381
- rule via_min_size: 0.3556 -> 0.381
- board text added: "PAS Capstone ADC Board"
- board text added: "V1.0"

Commit message: Should be ready for production now.
Parts:
- removed the REF** at (123.2, 97.8)
- REF**: value (none) -> mountinghole
Other:
- board text added: "Photo-Acoustic Sensing 2015 Capstone Mark Murnane Brandon Quade Tyler Quade Mahesh Shirole"
Changed lines of the file:
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@@
 (kicad_pcb (version 4) (host pcbnew "(after 2015-mar-04 BZR unknown)-product")
   (general
-    (links 0)
+    (links 191)
     (no_connects 0)
     (area 74.854999 100.254999 113.105001 163.905001)
     (thickness 1.6)
-    (drawings 10)
+    (drawings 11)
     (tracks 1103)
     (zones 0)
-    (modules 103)
+    (modules 102)
     (nets 66)
   )
@@
     (visible_elements FFFFFFFF)
     (pcbplotparams
-      (layerselection 0x00030_80000001)
+      (layerselection 0x010f0_80000001)
       (usegerberextensions false)
       (excludeedgelayer true)
@@
       (psa4output false)
       (plotreference true)
-      (plotvalue true)
+      (plotvalue false)
       (plotinvisibletext false)
       (padsonsilk false)
@@
       (outputformat 1)
       (mirror false)
-      (drillshape 1)
+      (drillshape 0)
       (scaleselection 1)
-      (outputdirectory ""))
+      (outputdirectory "Fab Plots/Plot4/"))
   )
   (net 0 "")
@@
     (descr "Mounting hole, Befestigungsbohrung, 3mm, No Annular, Kein Restring,")
     (tags "Mounting hole, Befestigungsbohrung, 3mm, No Annular, Kein Restring,")
-    (fp_text reference REF** (at 0 -4.0005) (layer F.SilkS)
+    (fp_text reference REF** (at 0 -4.0005) (layer F.SilkS) hide
       (effects (font (size 1 1) (thickness 0.15)))
     )
-    (fp_text value MountingHole_3mm (at 1.00076 5.00126) (layer F.Fab)
+    (fp_text value MountingHole_3mm (at -16.51 1.905) (layer F.Fab)
       (effects (font (size 1 1) (thickness 0.15)))
     )
@@
     (descr "Mounting hole, Befestigungsbohrung, 3mm, No Annular, Kein Restring,")
     (tags "Mounting hole, Befestigungsbohrung, 3mm, No Annular, Kein Restring,")
-    (fp_text reference REF** (at 0 -4.0005) (layer F.SilkS)
+    (fp_text reference REF** (at 0 -4.0005) (layer F.SilkS) hide
       (effects (font (size 1 1) (thickness 0.15)))
     )
-    (fp_text value MountingHole_3mm (at 1.00076 5.00126) (layer F.Fab)
+    (fp_text value MountingHole_3mm (at 14.605 1.27) (layer F.Fab)
       (effects (font (size 1 1) (thickness 0.15)))
     )
@@
     (descr "Mounting hole, Befestigungsbohrung, 3mm, No Annular, Kein Restring,")
     (tags "Mounting hole, Befestigungsbohrung, 3mm, No Annular, Kein Restring,")
-    (fp_text reference REF** (at 0 -4.0005) (layer F.SilkS)
+    (fp_text reference REF** (at 0.635 -0.635) (layer F.SilkS) hide
       (effects (font (size 1 1) (thickness 0.15)))
     )
-    (fp_text value "" (at -10.16 -1.27) (layer F.Fab) hide
+    (fp_text value mountinghole (at 10.16 -1.27) (layer F.Fab) hide
       (effects (font (size 1 1) (thickness 0.15)))
     )
@@
     )
   )
-  (module Mounting_Holes:MountingHole_2-5mm (layer F.Cu)
-    (at 123.19 97.79)
-    (descr "Mounting hole, Befestigungsbohrung, 2,5mm, No Annular, Kein Restring,")
-    (tags "Mounting hole, Befestigungsbohrung, 2,5mm, No Annular, Kein Restring,")
-    (fp_text reference REF** (at 0 -3.50012) (layer F.SilkS)
-      (effects (font (size 1 1) (thickness 0.15)))
-    )
-    (fp_text value MountingHole_2-5mm (at 0.09906 3.59918) (layer F.Fab)
-      (effects (font (size 1 1) (thickness 0.15)))
-    )
-    (fp_circle (center 0 0) (end 2.49936 0) (layer Cmts.User) (width 0.381))
-    (pad 1 thru_hole circle (at 0 0) (size 2.49936 2.49936) (drill 2.49936) (layers))
-  )
   (module Mounting_Holes:MountingHole_3mm (layer F.Cu)
     (at 110.49 102.87)
     (descr "Mounting hole, Befestigungsbohrung, 3mm, No Annular, Kein Restring,")
     (tags "Mounting hole, Befestigungsbohrung, 3mm, No Annular, Kein Restring,")
-    (fp_text reference REF** (at 0 -4.0005) (layer F.SilkS)
+    (fp_text reference REF** (at 0 -0.635) (layer F.SilkS) hide
       (effects (font (size 1 1) (thickness 0.15)))
     )
-    (fp_text value MountingHole_3mm (at 1.00076 5.00126) (layer F.Fab) hide
+    (fp_text value MountingHole_3mm (at -15.875 -0.635) (layer F.Fab) hide
       (effects (font (size 1 1) (thickness 0.15)))
     )
@@
     (pad 1 thru_hole circle (at 0 0) (size 2.99974 2.99974) (drill 2.99974) (layers))
   )
+  (gr_text "Photo-Acoustic Sensing\n2015 Capstone\nMark Murnane\nBrandon Quade\nTyler Quade\nMahesh Shirole" (at 95.25 132.08 90) (layer B.SilkS)
+    (effects (font (size 2.54 2.54) (thickness 0.508)) (justify mirror))
+  )
   (gr_text V1.0 (at 102.235 104.14) (layer F.SilkS)

Commit message: Adjusted 3d models
Parts:
- added D3: D_Schottky, Diodes_ThroughHole:Diode_DO-41_SOD81_Horizontal_RM10, F.Cu at (110.5, 128.3)
